File: KiCad/Row_A.sch (KiCad schematic (older format))
At the start: 37 parts, among them U101 RGB_WS2811, U102 RGB_WS2811, U103 RGB_WS2811, U104 RGB_WS2811, U105 RGB_WS2811, U106 RGB_WS2811, U107 RGB_WS2811, U108 RGB_WS2811, U109 RGB_WS2811, U110 RGB_WS2811, U111 RGB_WS2811, U112 RGB_WS2811, U113 RGB_WS2811, U114 RGB_WS2811, U115 RGB_WS2811, U116 RGB_WS2811

Commit message: building a Mood Lamp, in faricate directory
Parts:
- C101, C102, C103, C104, C105, C106, C107, C108, C109, C110, C111, C112, C113, C114, C115, C116: footprint c_0805 -> TiM:c_0805
- C117: footprint c_2917 -> TiM:c_2917
- S101, S102, S103, S104: footprint Screw -> TiM:Screw
- U101, U102, U103, U104, U105, U106, U107, U108, U109, U110, U111, U112, U113, U114, U115, U116: footprint RGB_WS2811 -> TiM:RGB_WS2811
