File: KiCad/Row_B.sch (KiCad schematic (older format))
At the start: 33 parts, among them U201 RGB_WS2811, U202 RGB_WS2811, U203 RGB_WS2811, U204 RGB_WS2811, U205 RGB_WS2811, U206 RGB_WS2811, U207 RGB_WS2811, U208 RGB_WS2811, U209 RGB_WS2811, U210 RGB_WS2811, U211 RGB_WS2811, U212 RGB_WS2811, U213 RGB_WS2811, U214 RGB_WS2811, U215 RGB_WS2811, U216 RGB_WS2811

Commit message: building a Mood Lamp, in faricate directory
Parts:
- C201, C202, C203, C204, C205, C206, C207, C208, C209, C210, C211, C212, C213, C214, C215, C216: footprint c_0805 -> TiM:c_0805
- C217: footprint c_2917 -> TiM:c_2917
- U201, U202, U203, U204, U205, U206, U207, U208, U209, U210, U211, U212, U213, U214, U215, U216: footprint RGB_WS2811 -> TiM:RGB_WS2811
