File: KiCad/Row_C.sch (KiCad schematic (older format))
At the start: 33 parts, among them U301 RGB_WS2811, U302 RGB_WS2811, U303 RGB_WS2811, U304 RGB_WS2811, U305 RGB_WS2811, U306 RGB_WS2811, U307 RGB_WS2811, U308 RGB_WS2811, U309 RGB_WS2811, U310 RGB_WS2811, U311 RGB_WS2811, U312 RGB_WS2811, U313 RGB_WS2811, U314 RGB_WS2811, U315 RGB_WS2811, U316 RGB_WS2811

Commit message: building a Mood Lamp, in faricate directory
Parts:
- C301, C302, C303, C304, C305, C306, C307, C308, C309, C310, C311, C312, C313, C314, C315, C316: footprint c_0805 -> TiM:c_0805
- C317: footprint c_2917 -> TiM:c_2917
- U301, U302, U303, U304, U305, U306, U307, U308, U309, U310, U311, U312, U313, U314, U315, U316: footprint RGB_WS2811 -> TiM:RGB_WS2811
