File: KiCad/Row_D.sch (KiCad schematic (older format))
At the start: 37 parts, among them U401 RGB_WS2811, U402 RGB_WS2811, U403 RGB_WS2811, U404 RGB_WS2811, U405 RGB_WS2811, U406 RGB_WS2811, U407 RGB_WS2811, U408 RGB_WS2811, U409 RGB_WS2811, U410 RGB_WS2811, U411 RGB_WS2811, U412 RGB_WS2811, U413 RGB_WS2811, U414 RGB_WS2811, U415 RGB_WS2811, U416 RGB_WS2811

Commit message: building a Mood Lamp, in faricate directory
Parts:
- C401, C402, C403, C404, C405, C406, C407, C408, C409, C410, C411, C412, C413, C414, C415, C416: footprint c_0805 -> TiM:c_0805
- C417: footprint c_2917 -> TiM:c_2917
- S401, S402, S403, S404: footprint Screw -> TiM:Screw
- U401, U402, U403, U404, U405, U406, U407, U408, U409, U410, U411, U412, U413, U414, U415, U416: footprint RGB_WS2811 -> TiM:RGB_WS2811
