File: KiCad/Row_E.sch (KiCad schematic (older format))
At the start: 37 parts, among them U501 RGB_WS2811, U502 RGB_WS2811, U503 RGB_WS2811, U504 RGB_WS2811, U505 RGB_WS2811, U506 RGB_WS2811, U507 RGB_WS2811, U508 RGB_WS2811, U509 RGB_WS2811, U510 RGB_WS2811, U511 RGB_WS2811, U512 RGB_WS2811, U513 RGB_WS2811, U514 RGB_WS2811, U515 RGB_WS2811, U516 RGB_WS2811

Commit message: building a Mood Lamp, in faricate directory
Parts:
- C501, C502, C503, C504, C505, C506, C507, C508, C509, C510, C511, C512, C513, C514, C515, C516: footprint c_0805 -> TiM:c_0805
- C517: footprint c_2917 -> TiM:c_2917
- S501, S502, S503, S504: footprint Screw -> TiM:Screw
- U501, U502, U503, U504, U505, U506, U507, U508, U509, U510, U511, U512, U513, U514, U515, U516: footprint RGB_WS2811 -> TiM:RGB_WS2811
