File: KiCad/Row_F.sch (KiCad schematic (older format))
At the start: 33 parts, among them U601 RGB_WS2811, U602 RGB_WS2811, U603 RGB_WS2811, U604 RGB_WS2811, U605 RGB_WS2811, U606 RGB_WS2811, U607 RGB_WS2811, U608 RGB_WS2811, U609 RGB_WS2811, U610 RGB_WS2811, U611 RGB_WS2811, U612 RGB_WS2811, U613 RGB_WS2811, U614 RGB_WS2811, U615 RGB_WS2811, U616 RGB_WS2811

Commit message: building a Mood Lamp, in faricate directory
Parts:
- C601, C602, C603, C604, C605, C606, C607, C608, C609, C610, C611, C612, C613, C614, C615, C616: footprint c_0805 -> TiM:c_0805
- C617: footprint c_2917 -> TiM:c_2917
- U601, U602, U603, U604, U605, U606, U607, U608, U609, U610, U611, U612, U613, U614, U615, U616: footprint RGB_WS2811 -> TiM:RGB_WS2811
