File: KiCad/Row_G.sch (KiCad schematic (older format))
At the start: 33 parts, among them U701 RGB_WS2811, U702 RGB_WS2811, U703 RGB_WS2811, U704 RGB_WS2811, U705 RGB_WS2811, U706 RGB_WS2811, U707 RGB_WS2811, U708 RGB_WS2811, U709 RGB_WS2811, U710 RGB_WS2811, U711 RGB_WS2811, U712 RGB_WS2811, U713 RGB_WS2811, U714 RGB_WS2811, U715 RGB_WS2811, U716 RGB_WS2811

Commit message: building a Mood Lamp, in faricate directory
Parts:
- C701, C702, C703, C704, C705, C706, C707, C708, C709, C710, C711, C712, C713, C714, C715, C716: footprint c_0805 -> TiM:c_0805
- C717: footprint c_2917 -> TiM:c_2917
- U701, U702, U703, U704, U705, U706, U707, U708, U709, U710, U711, U712, U713, U714, U715, U716: footprint RGB_WS2811 -> TiM:RGB_WS2811
