File: KiCad/Row_H.sch (KiCad schematic (older format))
At the start: 37 parts, among them U801 RGB_WS2811, U802 RGB_WS2811, U803 RGB_WS2811, U804 RGB_WS2811, U805 RGB_WS2811, U806 RGB_WS2811, U807 RGB_WS2811, U808 RGB_WS2811, U809 RGB_WS2811, U810 RGB_WS2811, U811 RGB_WS2811, U812 RGB_WS2811, U813 RGB_WS2811, U814 RGB_WS2811, U815 RGB_WS2811, U816 RGB_WS2811

Commit message: building a Mood Lamp, in faricate directory
Parts:
- C801, C802, C803, C804, C805, C806, C807, C808, C809, C810, C811, C812, C813, C814, C815, C816: footprint c_0805 -> TiM:c_0805
- C817: footprint c_2917 -> TiM:c_2917
- S801, S802, S803, S804: footprint Screw -> TiM:Screw
- U801, U802, U803, U804, U805, U806, U807, U808, U809, U810, U811, U812, U813, U814, U815, U816: footprint RGB_WS2811 -> TiM:RGB_WS2811
