File: KiCad/TiM.sch (KiCad schematic (older format))
At the start: 34 parts, among them P101 PWR_NW, P102 DO_N1, P103 DO_N2, P104 DI_N1, P105 DI_N2, P106 PWR_NE, P107 PWR_W, P108 PWR_E, P109 DI_W2, P110 DO_E2, P111 DI_W1, P112 DO_E1, P113 PWR_SW, P114 DI_S1, P115 DI_S2, P116 DO_S1, P117 DO_S2, P118 PWR_SE, P119 DO_H_SER, P120 DI_A_SER, P121 DI_A_SER, P122 DO_H_SER, P123 DI_A_Ser, P124 DO_H_Ser, P125 G>H, P126 F>G, P127 E>F, P128 D>E, P129 C>D, P130 B>C, P131 A>B

Commit message: building a Mood Lamp, in faricate directory
Parts:
- removed PCB101: CONN_1, PCB, symbol CONN_1
- L101: footprint OSHW_6mm -> TiM:OSHW_6mm
- L102: footprint Logo-WL3 -> TiM:Logo-WL3; manf# (none) -> mfr_pn
- P101, P106, P108, P119, P122: footprint SIL-PWR-2 -> TiM:SIL-PWR-2
- P102, P103, P110, P112, P116, P117: footprint CONN_S -> TiM:CONN_S
- P104, P105, P109, P111, P114, P115: footprint CONN_N -> TiM:CONN_N
- P107, P113, P118, P121, P123: footprint SIL-PWR -> TiM:SIL-PWR
- P120: footprint SIL-PWR-2 -> TiM:SIL-PWR
- P124: footprint SIL-PWR -> TiM:SIL-PWR-2
- P125, P126, P127, P128, P129, P130, P131: footprint ShortLink2 -> TiM:ShortLink2
Connections:
- no-connect marks 3 -> 2
